File: pcb/RescueAVR.kicad_pcb (KiCad board)
At the start: 2 copper layers, 68.6 x 53.3 mm, 24 parts, among them J1 Power, J2 Digital/PWM, J3 Analog, J4 Digital/PWM, J5 Conn_01x20_Socket, J6 Conn_01x08_Socket, Q1 BC547(NPN), Q2 BC557(PNP), U1 ATTinyX8,, U2 ATtinyX4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

Commit message: V2.6.0 and new PCBs
Parts:
- J1, J4: footprint Connector_PinSocket_2.54mm:PinSocket_1x08_P2.54mm_Vertical -> Connector_PinHeader_2.54mm:PinHeader_1x08_P2.54mm_Vertical; moved to B.Cu
- J2: footprint Connector_PinSocket_2.54mm:PinSocket_1x10_P2.54mm_Vertical -> Connector_PinHeader_2.54mm:PinHeader_1x10_P2.54mm_Vertical; moved to B.Cu
- J3: footprint Connector_PinSocket_2.54mm:PinSocket_1x06_P2.54mm_Vertical -> Connector_PinHeader_2.54mm:PinHeader_1x06_P2.54mm_Vertical; moved to B.Cu
- U1: value ATTinyX8, -> ATtinyX8
- U3: value ATtinyX2, X5, 1X, -> ATtiny11, 12, 13, 22, X5,
- turned J1 to -90 degrees
- turned J2 to -90 degrees
- turned J3 to -90 degrees
- turned J4 to -90 degrees
Connections:
- J1 pad 2: /IOREF -> unconnected-(J1-Pin_2-Pad2)
- J1 pad 3: /~{RESET} -> unconnected-(J1-Pin_3-Pad3)
- J2 pad 3: /AREF -> unconnected-(J2-Pin_3-Pad3)
- J4 pad 7: /TX/1 -> unconnected-(J4-Pin_7-Pad7)
- J4 pad 8: /RX/0 -> unconnected-(J4-Pin_8-Pad8)
Other:
- board text added: "+"
- board text added: "-"
- board text added: "12V"
- board text added: "5V"
- board text added: "Booster"
- board text added: "RescueAVR V1.1"
- board text removed: "RescueAVR V1.0"
