File: pcb/RescueAVR.kicad_sch (KiCad schematic)
At the start: 20 parts, among them J1 Power, J2 Digital/PWM, J3 Analog, J4 Digital/PWM, J5 Conn_01x20_Socket, J6 Conn_01x08_Socket, Q1 BC547(NPN), Q2 BC557(PNP), U1 ATmegaX8, U2 ATtinyX4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

Commit message: V2.6.0 and new PCBs
Parts:
- J1, J4: footprint Connector_PinSocket_2.54mm:PinSocket_1x08_P2.54mm_Vertical -> Connector_PinHeader_2.54mm:PinHeader_1x08_P2.54mm_Vertical
- J2: footprint Connector_PinSocket_2.54mm:PinSocket_1x10_P2.54mm_Vertical -> Connector_PinHeader_2.54mm:PinHeader_1x10_P2.54mm_Vertical
- J3: footprint Connector_PinSocket_2.54mm:PinSocket_1x06_P2.54mm_Vertical -> Connector_PinHeader_2.54mm:PinHeader_1x06_P2.54mm_Vertical
- U1: value ATmegaX8 -> ATtinyX8
- U3: value ATtinyX5, ATtiny1X -> ATtiny11, 12, 13, 22, X5,
Changed lines of the file:
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@@
 	(title_block
 		(title "RescueAVR")
-		(date "2024-08-25")
-		(rev "1.0")
+		(date "2024-09-06")
+		(rev "1.1")
 		(company "Arduino Craft Corner")
 	)
@@
 			)
 		)
-		(property "Footprint" "Connector_PinSocket_2.54mm:PinSocket_1x08_P2.54mm_Vertical"
+		(property "Footprint" "Connector_PinHeader_2.54mm:PinHeader_1x08_P2.54mm_Vertical"
 			(at 39.37 39.37 0)
 			(effects
@@
 			)
 		)
-		(property "Footprint" "Connector_PinSocket_2.54mm:PinSocket_1x10_P2.54mm_Vertical"
+		(property "Footprint" "Connector_PinHeader_2.54mm:PinHeader_1x10_P2.54mm_Vertical"
 			(at 57.15 36.83 0)
 			(effects
@@
 			)
 		)
-		(property "Footprint" "Connector_PinSocket_2.54mm:PinSocket_1x06_P2.54mm_Vertical"
+		(property "Footprint" "Connector_PinHeader_2.54mm:PinHeader_1x06_P2.54mm_Vertical"
 			(at 39.37 64.77 0)
 			(effects
@@
 			)
 		)
-		(property "Footprint" "Connector_PinSocket_2.54mm:PinSocket_1x08_P2.54mm_Vertical"
+		(property "Footprint" "Connector_PinHeader_2.54mm:PinHeader_1x08_P2.54mm_Vertical"
 			(at 57.15 67.31 0)
 			(effects
@@
 			)
 		)
-		(property "Value" "ATmegaX8"
+		(property "Value" "ATtinyX8"
 			(at 107.95 96.52 0)
 			(effects
@@
 			)
 		)
-		(property "Value" "ATtinyX5, ATtiny1X"
+		(property "Value" "ATtiny11, 12, 13, 22, X5,"
 			(at 223.52 52.07 0)
 			(effects
