File: pcb/RescueAVRAdapter.kicad_pcb (KiCad board)
At the start: 2 copper layers, 68.6 x 53.3 mm, 12 parts, among them J5 Conn_01x20_Socket, J6 Conn_01x08_Socket, U1 ATmega16A-P, U2 ATmega162-16P, U3 ATtiny2313-20P, U4 ATtiny861-20P

Commit message: V2.6.0 and new PCBs
Parts:
- removed MH1, MH2, MH3, MH4: MountingHole_3.2mm, Arduino_MountingHole:MountingHole_3.2mm
- J5: footprint Connector_PinSocket_2.54mm:PinSocket_1x20_P2.54mm_Vertical -> Connector_PinHeader_2.54mm:PinHeader_1x20_P2.54mm_Vertical; moved to B.Cu
- J6: footprint Connector_PinSocket_2.54mm:PinSocket_1x08_P2.54mm_Vertical -> Connector_PinHeader_2.54mm:PinHeader_1x08_P2.54mm_Vertical; moved to B.Cu
- U1, U2: footprint Package_DIP:DIP-40_W15.24mm -> Package_DIP:DIP-40_W15.24mm_Socket
- U3, U4: footprint Package_DIP:DIP-20_W7.62mm -> Package_DIP:DIP-20_W7.62mm_Socket
- turned J5 to 90 degrees
- turned J6 to 90 degrees
Other:
- board text added: "RescueAVR Adapter V1.2"
- board text removed: "RescueAVR Adapter V1.1"
